File: L Smart Baton/L Smart Baton.kicad_sch (KiCad schematic)
At the start: 51 parts, among them J1 USB4105-GF-A, SW1 B3U-1000P, SW1_R1 1k, U1 MDBT50Q-1MV2, U2 LSM6DSOX, U3 BQ24074RGT, U4 TPS63001

Commit message: Final PCB layout
Parts:
- C1, C2, C_BAT_BQ1, C_IN_BQ1, C_IN_TPS1, C_LFXO1, C_LFXO2, C_MCU_100N1, C_MCU_BULK1, C_OUT_BQ1, C_SENSE1, C_TPS_OUT1, C_TPS_OUT2, D1, R1, R2, R3, R4, R5, RGB_BLUE_R1, RGB_GREEN_R1, RGB_RED_R1, R_BOT1, R_CHG_PULLUP1, R_EN2, R_ILIM1, R_ISET1, R_ITERM1, R_TMR1, R_TOP1, R_TS1, R_VINA1, VINA_C1: KiLib_Generator (none) -> SMD_2terminal_chip_molded
- J_BAT1: KiLib_Generator (none) -> connector/JST
- J_SWD1: KiLib_Generator (none) -> connector/pin_header_socket
- L1: KiLib_Generator (none) -> inductor/SMD
- SW1_R1: footprint (none) -> Resistor_SMD:R_0603_1608Metric; KiLib_Generator (none) -> SMD_2terminal_chip_molded
- U3: KiLib_Generator (none) -> package/no_lead
Connections:
- net BLE_LED: now also U1.22 (P0.06); no longer U1.43 (P0.21)
- net RGB_BLUE: now also U1.49 (P0.25); no longer U1.48 (P0.24)
- net RGB_RED: now also U1.47 (P1.00); no longer U1.46 (P0.22)
- no-connect marks 47 -> 50
