File: L Smart Baton/L Smart Baton.kicad_sch (KiCad schematic)
At the start: 50 parts, among them J1 USB4105-GF-A, SW1 B3U-1000P, U1 MDBT50Q-1MV2, U2 LSM6DSOX, U3 BQ24074RGT, U4 TPS63001

Commit message: add 1k resistor to button
Parts:
- added SW1_R1: 1k, symbol Device:R
Connections:
- net USER_BTN: now also SW1_R1.1; no longer SW1.1
- new net: SW1.1, SW1_R1.2
Changed lines of the file:
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@@
 	(wire
 		(pts
-			(xy 185.42 361.95) (xy 203.2 361.95)
+			(xy 176.53 361.95) (xy 190.5 361.95)
 		)
 		(stroke
@@
 	(wire
 		(pts
+			(xy 198.12 361.95) (xy 203.2 361.95)
+		)
+		(stroke
+			(width 0)
+			(type default)
+		)
+	)
+	(wire
+		(pts
 			(xy 248.92 269.24) (xy 261.62 269.24)
 		)
@@
 	)
 	(label "USER_BTN"
-		(at 185.42 361.95 0)
+		(at 176.53 361.95 0)
 		(effects
 			(font
@@
 					(unit 1)
 				)
+			)
+		)
+	)
+	(symbol
+		(lib_id "Device:R")
+		(at 194.31 361.95 90)
+		(unit 1)
+		(body_style 1)
+		(exclude_from_sim no)
+		(in_bom yes)
+		(on_board yes)
+		(in_pos_files yes)
+		(dnp no)
+		(fields_autoplaced yes)
+		(property "Reference" "SW1_R1"
+			(at 194.31 355.6 90)
+			(show_name no)
+			(do_not_autoplace no)
+			(effects
+				(font
+					(size 1.27 1.27)
+				)
+			)
+		)
+		(property "Value" "1k"
+			(at 194.31 358.14 90)
+			(show_name no)
+			(do_not_autoplace no)
+			(effects
+				(font
+					(size 1.27 1.27)
+				)
+			)
+		)
+		(property "Footprint" ""
+			(at 194.31 363.728 90)
+			(hide yes)
+			(show_name no)
+			(do_not_autoplace no)
+			(effects
+				(font
+					(size 1.27 1.27)
+				)
+			)
+		)
+		(property "Datasheet" ""
+			(at 194.31 361.95 0)
+			(hide yes)
+			(show_name no)
+			(do_not_autoplace no)
+			(effects
+				(font
+					(size 1.27 1.27)
+				)
+			)
+		)
+		(property "Description" "Resistor"
+			(at 194.31 361.95 0)
+			(hide yes)
+			(show_name no)
+			(do_not_autoplace no)
+			(effects
+				(font
+					(size 1.27 1.27)
+				)
+			)
+		)
+		(pin "2"
+		)
+		(pin "1"
+		)
+		(instances
+			(project "L Smart Baton"
+				(path "/0317b452-a1b7-45b1-86f0-abd0d959d24f"
+					(reference "SW1_R1")
+					(unit 1)
+				)

Commit message: Add files via upload
Parts:
- C1, C2, C_BAT_BQ1, C_IN_BQ1, C_IN_TPS1, C_LFXO1, C_LFXO2, C_MCU_100N1, C_MCU_BULK1, C_OUT_BQ1, C_SENSE1, C_TPS_OUT1, C_TPS_OUT2, D1, R1, R2, R3, R4, R5, RGB_BLUE_R1, RGB_GREEN_R1, RGB_RED_R1, R_BOT1, R_CHG_PULLUP1, R_EN2, R_ILIM1, R_ISET1, R_ITERM1, R_TMR1, R_TOP1, R_TS1, R_VINA1, VINA_C1: KiLib_Generator (none) -> SMD_2terminal_chip_molded
- J_BAT1: KiLib_Generator (none) -> connector/JST
- J_SWD1: KiLib_Generator (none) -> connector/pin_header_socket
- L1: KiLib_Generator (none) -> inductor/SMD
- SW1_R1: footprint (none) -> Resistor_SMD:R_0603_1608Metric; KiLib_Generator (none) -> SMD_2terminal_chip_molded
- U3: KiLib_Generator (none) -> package/no_lead
Connections:
- net BLE_LED: now also U1.22 (P0.06); no longer U1.43 (P0.21)
- net RGB_BLUE: now also U1.49 (P0.25); no longer U1.48 (P0.24)
- net RGB_RED: now also U1.47 (P1.00); no longer U1.46 (P0.22)
