File: L Smart Baton/L Smart Baton.kicad_sch (KiCad schematic)
At the start: 51 parts, among them J1 USB4105-GF-A, SW1 B3U-1000P, SW1_R1 1k, U1 MDBT50Q-1MV2, U2 LSM6DSOX, U3 BQ24074RGT, U4 TPS63001

Commit message: Changed unavailable components with substitute pads. FINAL DRAFT
Parts:
- J1: value USB4105-GF-A -> TYPEC-304A-ACP16W
- L1: value 74438335022 -> MPN3015S2R2MT; footprint Inductor_SMD:L_Wuerth_MAPI-3015 -> Inductor_SMD:L_Sunlord_SWPA3015S
Changed lines of the file:
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@@
 			)
 		)
-		(property "Value" "USB4105-GF-A"
+		(property "Value" "TYPEC-304A-ACP16W"
 			(at 304.8 105.4099 90)
 			(show_name no)
@@
 			)
 		)
-		(property "Datasheet" "https://gct.co/files/drawings/usb4105.pdf"
+		(property "Datasheet" ""
 			(at 285.75 107.95 0)
 			(hide yes)
@@
 			)
 		)
-		(property "Value" "74438335022"
+		(property "Value" "MPN3015S2R2MT"
 			(at 266.954 237.998 0)
 			(show_name no)
@@
 			)
 		)
-		(property "Footprint" "Inductor_SMD:L_Wuerth_MAPI-3015"
+		(property "Footprint" "Inductor_SMD:L_Sunlord_SWPA3015S"
 			(at 269.24 228.6 0)
 			(hide yes)
@@
 			)
 		)
-		(property "Datasheet" "https://www.we-online.com/en/components/products/WE-MAPI?utm_source=chatgpt.com"
+		(property "Datasheet" ""
 			(at 269.24 228.6 0)
 			(hide yes)
